File: Circuit 8/Circuit 8/Circuit 8.kicad_sch (KiCad schematic)
At the start: 37 parts, among them SW1 RIGHT, SW2 LEFT, SW3 LEFT, U1 74LS14, U10 HDSP-7803, U11 HDSP-7803, U12 74LS08, U13 74LS08, U14 74LS04, U15 74LS04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

Commit message: Add files via upload
Connections:
- net at U16.3, U6.5 (Q), U8.2 (C): no longer U15.3, U5.9 (Q), U8.1 (B)
- new net: U15.3, U5.9 (Q), U8.1 (B)
Other:
- note added: "Player 1"
- note added: "Player 2"
- note added: "Reset"
- moved on the sheet: C3, R5, R6, SW3, U2B
