File: Circuit 1/Circuit 1/Circuit 1.kicad_sch (KiCad schematic)
At the start: 18 parts, among them SW1 SW_DIP_x08, SW2 SW_DIP_x08, U1 7408, U2 7485, U3 7432

Commit message: Add files via upload
Parts:
- removed U1: 7408, symbol 74xx_IEEE:7408
- removed U2: 7485, symbol 74xx_IEEE:7485
- removed U3: 7432, symbol 74xx_IEEE:7432
- added R14: 220, symbol Device:R_US
- added U1, U5, U6, U7: 74LS08, symbol 74xx:74LS08
- added U2: 74LS85, symbol 74xx:74LS85
- R1, R12, R13, R2, R3, R4, R6, R7, R8, R9: value R_US -> 220
Connections:
- net GND: now also U2.2 (Ia<b), U2.4 (Ia>b), U2.8 (GND)
- net at D1.4 (BK): now also R14.2
- net at R8.2, SW2.14: now also U2.12 (A1)
- net at R12.1: now also U5.3
- net at R3.2, SW1.14: now also U2.11 (B1)
- net at R10.2, SW1.9: now also U1.1
- net at R5.2, SW2.9: now also U1.2
- net at R9.2, SW2.13: now also U2.10 (A0)
- net at R13.1: now also U7.3
- net at R4.2, SW1.13: now also U2.9 (B0)
- net at R6.2, SW2.16: now also U2.15 (A3)
- net at R1.2, SW1.16: now also U2.1 (B3)
- net at R7.2, SW2.15: now also U2.13 (A2)
- net at R2.2, SW1.15: now also U2.14 (B2)
- new net: R14.1, U6.3
- new net: U2.7 (Oa<b), U6.1
- new net: U1.3, U5.2, U6.2, U7.2
- new net: U2.6 (Oa=b), U5.1
- new net: U2.5 (Oa>b), U7.1
- new net VCC: U2.16 (VCC), U2.3 (Ia=b)
Other:
- note added: "Circuit 1: Guess the number"
- note removed: "Circuit 2: Guess the number"
- moved on the sheet: D1, R12, R13
